File: board/DuPal_DIP/DuPal_DIP.kicad_pcb (KiCad board)
At the start: 2 copper layers, 113 x 78.7 mm, 57 parts, among them J1 AVR-ISP-6, J2 RS232, J3 Power IN, SW1 SW_Push, SW2 Power, U1 ATmega8A-PU, U10 24 Pin PAL, U2 74HC595, U3 74HC595, U5 20 Pin PAL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

Commit message: Updated to KiCad 7
Connections:
- net /~PISO_CLR renamed /~{PISO_CLR}
- net /~RESET renamed /~{RESET}
- net /~SIPO_CLR renamed /~{SIPO_CLR}
- net /~SIPO_OE renamed /~{SIPO_OE}
Other:
- net class Default removed
- net class POWER removed

Commit message: Resolves DRC issues
Parts:
- renumbered G*** to G***2
Connections:
- J2 pad 1: Net-(J2-Pad1) -> unconnected-(J2-Pad1)
- J2 pad 6: Net-(J2-Pad6) -> unconnected-(J2-Pad6)
- J2 pad 7: Net-(J2-Pad7) -> unconnected-(J2-Pad7)
- J2 pad 8: Net-(J2-Pad8) -> unconnected-(J2-Pad8)
- J2 pad 9: Net-(J2-Pad9) -> unconnected-(J2-Pad9)
- J3 pad 3: (no net) -> unconnected-(J3-Pad3)
- SW2 pad 3: (no net) -> unconnected-(SW2-Pad3)
- U1 pad 13: Net-(U1-Pad13) -> unconnected-(U1-PD7-Pad13)
- U1 pad 25: Net-(U1-Pad25) -> unconnected-(U1-PC2-Pad25)
- U1 pad 26: Net-(U1-Pad26) -> unconnected-(U1-PC3-Pad26)
- U2 pad 1: /SIPO_O_2 -> unconnected-(U2-QB-Pad1)
- U2 pad 15: /SIPO_O_1 -> unconnected-(U2-QA-Pad15)
- U6 pad 14: Net-(U6-Pad14) -> unconnected-(U6-T1OUT-Pad14)
- U9 pad 9: Net-(U9-Pad9) -> unconnected-(U9-QH'-Pad9)

Commit message: Hides unconnected pins
Parts:
- Y1: value 8Mhz -> 20Mhz
Connections:
- U2 pad 1: unconnected-(U2-QB-Pad1) -> /SIPO_O_2
- U2 pad 15: unconnected-(U2-QA-Pad15) -> /SIPO_O_1
Changed lines of the file:
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@@
   (net 68 "/P24_14")
   (net 69 "/P24_23")
-  (net 70 "unconnected-(U2-QB-Pad1)")
+  (net 70 "/SIPO_O_2")
   (net 71 "/P20_9")
   (net 72 "/P20_11")
@@
   (net 80 "/P20_2")
   (net 81 "/P20_1")
-  (net 82 "unconnected-(U2-QA-Pad15)")
+  (net 82 "/SIPO_O_1")
   (net 83 "Net-(U3-QH')")
   (net 84 "unconnected-(U6-T1OUT-Pad14)")
@@
       (stroke (width 0.1) (type solid)) (layer "F.Fab"))
     (pad "1" thru_hole rect (at 0 0) (size 1.6 1.6) (drill 0.8) (layers "*.Cu" "*.Mask")
-      (net 70 "unconnected-(U2-QB-Pad1)") (pinfunction "QB") (pintype "tri_state+no_connect"))
+      (net 70 "/SIPO_O_2") (pinfunction "QB") (pintype "tri_state"))
     (pad "2" thru_hole oval (at 0 2.54) (size 1.6 1.6) (drill 0.8) (layers "*.Cu" "*.Mask")
       (net 69 "/P24_23") (pinfunction "QC") (pintype "tri_state"))
@@
       (net 52 "/SIPO_SER") (pinfunction "SER") (pintype "input"))
     (pad "15" thru_hole oval (at 7.62 2.54) (size 1.6 1.6) (drill 0.8) (layers "*.Cu" "*.Mask")
-      (net 82 "unconnected-(U2-QA-Pad15)") (pinfunction "QA") (pintype "tri_state+no_connect"))
+      (net 82 "/SIPO_O_1") (pinfunction "QA") (pintype "tri_state"))
     (pad "16" thru_hole oval (at 7.62 0) (size 1.6 1.6) (drill 0.8) (layers "*.Cu" "*.Mask")
       (net 10 "VCC") (pinfunction "VCC") (pintype "power_in"))
@@
         (effects (font (size 1 1) (thickness 0.15)))
     )
-    (fp_text value "8Mhz" (at 2.44 3.525 90) (layer "F.Fab")
+    (fp_text value "20Mhz" (at 2.44 3.525 90) (layer "F.Fab")
         (effects (font (size 1 1) (thickness 0.15)))
     )
